File: Karim_Arduino.sch (KiCad schematic (older format))
At the start: 30 parts, among them J1 ICSP, J2 Conn_01x15, J3 Conn_01x15, SW1 SW_Push, U1 ATMEGA328P_TQFP, U2 AMS1117-3.3

Commit message: Fix ERC Issues
-Power Flag
-Output pin of voltage regulator was connected to bidirectional pin of the micro controller.
Parts:
- U1: Field4 IC-09069 -> (none)
Changed lines of the file:
@@
 F 2 "Silicon-Standard:TQFP32-08" H 2950 7050 20  0001 C CNN
 F 3 "" H 2950 5700 50  0001 C CNN
-F 4 "IC-09069" H 2950 7031 60  0000 C CNN "Field4"
+F 4 "" H 2950 7031 60  0000 C CNN "Field4"
 	1    2950 5700
 	1    0    0    -1
@@
 Wire Wire Line
 	2150 1250 2150 1300
-Wire Wire Line
-	1700 1250 2150 1250
 Connection ~ 2150 1250
 Wire Wire Line
@@
 P 6650 3850
 F 0 "#PWR0102" H 6650 3700 50  0001 C CNN
-F 1 "VCC" H 6665 4023 50  0000 C CNN
+F 1 "VCC" V 6665 4023 50  0000 C CNN
 F 2 "" H 6650 3850 50  0001 C CNN
 F 3 "" H 6650 3850 50  0001 C CNN
@@
 Wire Wire Line
 	1350 4800 1350 4850
+$Comp
+L power:PWR_FLAG #FLG0101
+U 1 1 5FB47AAE
+P 2700 1850
+F 0 "#FLG0101" H 2700 1925 50  0001 C CNN
+F 1 "PWR_FLAG" H 2700 2023 50  0000 C CNN
+F 2 "" H 2700 1850 50  0001 C CNN
+F 3 "~" H 2700 1850 50  0001 C CNN
+	1    2700 1850
+	-1   0    0    1
+$EndComp
+$Comp
+L power:PWR_FLAG #FLG0102
+U 1 1 5FB47DC1
+P 1700 1400
+F 0 "#FLG0102" H 1700 1475 50  0001 C CNN
+F 1 "PWR_FLAG" H 1700 1573 50  0000 C CNN
+F 2 "" H 1700 1400 50  0001 C CNN
+F 3 "~" H 1700 1400 50  0001 C CNN
+	1    1700 1400
+	-1   0    0    1
+$EndComp
+Wire Wire Line
+	1700 1400 1700 1250
+Wire Wire Line
+	1700 1250 2150 1250
+Connection ~ 1700 1250
+Wire Wire Line
+	2700 1850 3000 1850
+Connection ~ 3000 1850
 $EndSCHEMATC

Commit message: Placing components on PCB
Parts:
- D2: value YELLOW -> BLUE
- J2, J3: footprint Connector_PinSocket_2.54mm:PinSocket_1x15_P2.54mm_Vertical -> Connector_PinHeader_2.54mm:PinHeader_1x15_P2.54mm_Vertical
Changed lines of the file:
@@
 P 4150 1400
 F 0 "D2" V 4196 1330 50  0000 R CNN
-F 1 "YELLOW" V 4105 1330 50  0000 R CNN
+F 1 "BLUE" V 4105 1330 50  0000 R CNN
 F 2 "LED_SMD:LED_0603_1608Metric" V 4150 1400 50  0001 C CNN
 F 3 "~" V 4150 1400 50  0001 C CNN
@@
 F 0 "J3" H 6850 4150 50  0000 L CNN
 F 1 "Conn_01x15" H 6750 4050 50  0000 L CNN
-F 2 "Connector_PinSocket_2.54mm:PinSocket_1x15_P2.54mm_Vertical" H 6850 3250 50  0001 C CNN
+F 2 "Connector_PinHeader_2.54mm:PinHeader_1x15_P2.54mm_Vertical" H 6850 3250 50  0001 C CNN
 F 3 "~" H 6850 3250 50  0001 C CNN
 	1    6850 3250
@@
 F 0 "J2" H 5250 2350 50  0000 C CNN
 F 1 "Conn_01x15" H 5300 2450 50  0000 C CNN
-F 2 "Connector_PinSocket_2.54mm:PinSocket_1x15_P2.54mm_Vertical" H 5200 3250 50  0001 C CNN
+F 2 "Connector_PinHeader_2.54mm:PinHeader_1x15_P2.54mm_Vertical" H 5200 3250 50  0001 C CNN
 F 3 "~" H 5200 3250 50  0001 C CNN
 	1    5200 3250
