File: Karim_Arduino.kicad_pcb (KiCad board)
At the start: 2 copper layers, 39.8 x 23.7 mm, 30 parts, among them J1 ICSP, J2 Conn_01x15, J3 Conn_01x15, SW1 SW_Push, U1 ATMEGA328P, U2 AMS1117-3.3

Commit message: Routing components
Parts:
- moved R3 19.1 mm to (124.2, 83.9), turned to 0 degrees
- moved HSE1 5.73 mm to (155.4, 96.2), turned to 270 degrees
- moved R9 4.16 mm to (138.4, 96.8), turned to 270 degrees
- moved R8 3.74 mm to (127.1, 93.2)
- moved C9 3.57 mm to (157.7, 95.9)
- moved R10 3.13 mm to (127.8, 95.5), turned to 0 degrees
- moved R6 2.84 mm to (131.7, 96.4)
- moved R5 2.75 mm to (138.4, 84.2)
- moved R1 2.36 mm to (127.2, 83.9), turned to 180 degrees
- moved C1 2.25 mm to (149.1, 88.2), turned to 45 degrees
- moved R7 1.87 mm to (134.7, 96.5), turned to 90 degrees
- moved C6 0.85 mm to (133.3, 84.6)
- moved C8 0.75 mm to (153.1, 95.9), turned to 270 degrees
- moved C7 0.71 mm to (134.4, 84.6)
- moved J1 0.70 mm to (121.8, 87.7)
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Routing:
- net VCC: track 0.00 -> 90.1 mm, vias 0 -> 4
- net RESET: track 0.00 -> 68.1 mm, vias 0 -> 2
- net MISO: track 0.00 -> 42.3 mm, vias 0 -> 1
- net SCK: track 0.00 -> 42.1 mm, vias 0 -> 2
- net MOSI: track 0.00 -> 40.7 mm, vias 0 -> 2
- net TXO: track 0.00 -> 26.7 mm, vias 0 -> 3
- net Net-(C9-Pad1): track 0.00 -> 23.5 mm, vias 0 -> 2
- net RXI: track 0.00 -> 22.7 mm, vias 0 -> 3
- net A6: track 0.00 -> 17.8 mm, vias 0 -> 1
- net A7: track 0.00 -> 16.2 mm, vias 0 -> 1
- net HSE_IN: track 0.00 -> 14.9 mm, vias 0 -> 2
- net D2: track 0.00 -> 14.0 mm
- net VIN: track 0.00 -> 13.7 mm, vias 0 -> 1
- net Net-(J2-Pad14): track 0.00 -> 12.3 mm
- net D10: track 0.00 -> 11.7 mm
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Other:
- rule via_min_size: 0.6 -> 0.45
