File: Karim_Arduino.kicad_pcb (KiCad board)
At the start: 2 copper layers, 39.8 x 23.7 mm, 30 parts, among them J1 ICSP, J2 Conn_01x15, J3 Conn_01x15, SW1 SW_Push, U1 ATMEGA328P, U2 AMS1117-3.3

Commit message: Update Footprints positions
Other:
- board text added: "DESIGNED BY: KARIM BOUANANE"
- board text added: "El Mardi Imane: "si tu veux tu peux""
